File: noname.kicad_pcb (KiCad board)
At the start: 2 copper layers, 27.9 x 31.8 mm, 23 parts, among them J1 USB_B_Micro, J2 Micro_SD_Card_Det, J3 Conn_01x01_Male, J4 Conn_01x01_Male, U1 BL652, U2 ADP2302ARDZ-3.3

Commit message: final changes
Parts:
- removed CSS2: 10u, Resistor_SMD:R_1210_3225Metric_Pad1.42x2.65mm_HandSolder
- removed J3, J4, SWDCLK, SWDIO, VIO, nRESET: Conn_01x01_Male, Connector_PinHeader_1.00mm:PinHeader_1x01_P1.00mm_Vertical
- removed TP2, TP4, TP6: TestPoint, TestPoint:TestPoint_THTPad_1.0x1.0mm_Drill0.5mm
- added 3.3V: Conn_01x01_Male, Connector_PinHeader_1.00mm:PinHeader_1x01_P1.00mm_Vertical, F.Cu at (146.2, 54.0)
- added G***: LOGO, logos:bac-logo, F.Cu at (132.3, 70.9)
- added MOSI: TestPoint, TestPoint:TestPoint_THTPad_1.0x1.0mm_Drill0.5mm, F.Cu at (145.4, 50.9)
- added PGOOD: TestPoint, TestPoint:TestPoint_THTPad_1.0x1.0mm_Drill0.5mm, F.Cu at (150.9, 64.1)
- added SCLK: TestPoint, TestPoint:TestPoint_THTPad_1.0x1.0mm_Drill0.5mm, F.Cu at (128.5, 55.6)
- moved GND 1.37 mm to (150.2, 55.0)
- moved MISO 1.35 mm to (145.4, 48.8)
Connections:
- J2 pad 2: /CS -> GND
- U1 pad 4: /CS -> GND
- U1 pad 5: /SWDIO -> Net-(U1-Pad5)
- U1 pad 6: /SWDCLK -> Net-(U1-Pad6)
- U1 pad 7: /nRESET -> Net-(U1-Pad7)
Routing:
- net /CS: track 36.8 -> 0.00 mm, vias 2 -> 0
- net GND: track 54.4 -> 67.1 mm, vias 8 -> 12
- net /nRESET: track 9.24 -> 0.00 mm
- net /SWDIO: track 8.87 -> 0.00 mm
- net /SWDCLK: track 8.37 -> 0.00 mm
- net /VIO: track 5.87 -> 0.00 mm
- net /PGOOD: track 7.81 -> 2.93 mm
- net /MOSI: track 40.5 -> 39.4 mm
- net /MISO: track 28.9 -> 27.9 mm
Other:
- board size 27.9 x 31.8 mm -> 25.4 x 31.8 mm
