File: old_schematic.sch (KiCad schematic (older format))
At the start: 23 parts, among them J1 USB_B_Micro, J10 Conn_01x01_Male, J2 Micro_SD_Card_Det, J3 Conn_01x01_Male, J4 Conn_01x01_Male, J6 Conn_01x01_Male, J7 Conn_01x01_Male, J8 Conn_01x01_Male, J9 Conn_01x01_Male, U1 BL652, U2 ADP2302ARDZ-3.3

Commit message: final changes
Parts:
- removed CSS2: 10u, Resistor_SMD:R_1210_3225Metric_Pad1.42x2.65mm_HandSolder, symbol Device:C_Small
- removed J10, J6, J7, J8, J9: Conn_01x01_Male, Connector_PinHeader_1.00mm:PinHeader_1x01_P1.00mm_Vertical, symbol Connector:Conn_01x01_Male
- added C1: 470n, Capacitor_SMD:C_0805_2012Metric_Pad1.15x1.40mm_HandSolder, symbol Device:C_Small
- added C2: 4.7u, Capacitor_SMD:C_0805_2012Metric_Pad1.15x1.40mm_HandSolder, symbol Device:C_Small
- added U3: MSP430FR5720IRGE, Package_DFN_QFN:Texas_S-PVQFN-N24_EP2.1x2.1mm, symbol MCU_Texas_MSP430:MSP430FR5720IRGE
Connections:
- net labels removed: SWDCLK, SWDIO, VIO, nRESET
- wire segments 54 -> 50
Other:
- moved on the sheet: J2, TP3, TP4, TP6, U1
